File: Lab2_starter.kicad_pcb (KiCad board)
At the start: 4 copper layers, 139.7 x 101.6 mm, 77 parts, among them J1 973582101, J10 Conn_01x02, J11 Conn_01x02, J12 Conn_01x02, J13 Conn_01x02, J14 Conn_01x02, J15 Conn_01x02, J16 Conn_01x02, J2 973582100, J3 973582101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

Commit message: Final Board Revision YAY
Parts:
- C19, C4, Dboot1, Rboot1: moved to F.Cu
- U1: moved to B.Cu
- moved J12 30.2 mm to (79.2, 109.8), turned to 90 degrees
- moved J9 27.7 mm to (59.1, 136.9), turned to -90 degrees
- moved J10 27.0 mm to (67.6, 136.9), turned to -90 degrees
- moved J8 22.3 mm to (66.7, 115.2), turned to 90 degrees
- moved J5 19.0 mm to (63.2, 136.1)
- moved U1 14.5 mm to (72.2, 133.8), turned to 90 degrees
- moved R4 13.3 mm to (67.7, 132.6)
- moved R3 12.8 mm to (69.0, 118.6), turned to 180 degrees
- moved C16 9.96 mm to (51.1, 121.7)
- moved C19 9.64 mm to (81.7, 122.0), turned to -90 degrees
- moved C3 8.86 mm to (69.7, 122.0), turned to -90 degrees
- moved Dboot1 8.23 mm to (74.4, 122.0), turned to -90 degrees
- moved C4 7.94 mm to (74.3, 130.3), turned to -90 degrees
- moved C12 4.68 mm to (63.1, 128.1)
- moved C15 4.68 mm to (63.1, 130.2)
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Routing:
- net GND: track 9.96 -> 26.3 mm
- net Vsw: track 31.3 -> 22.6 mm
- net C2000 D': track 119.0 -> 127.2 mm
- net D': track 16.7 -> 9.28 mm
- net C2000 D : track 114.3 -> 120.8 mm
- net D: track 19.4 -> 12.9 mm
- net +12V: track 87.0 -> 91.4 mm
- net Vin_sens: track 36.9 -> 33.2 mm
- net /ADCINA4: track 7.87 -> 4.56 mm
- net Vboot: track 14.9 -> 17.8 mm
- net Net-(U1-HO): track 4.96 -> 2.27 mm
- net I_L: track 42.1 -> 42.9 mm
- net Vout: track 23.3 -> 22.7 mm
- added copper zone on In2.Cu, net Vsw
